File: Electronic Stuff/IR Module V2/IR_module_V0_2.brd (EAGLE design)
At the start: 100 x 80 mm, 24 parts, among them IC1 74HCT02N, Q1 IRF540, T1 2N3904

Commit message: IR module V0.2
Parts:
- removed JP2: (no value), jumper:JP2
- removed JP6: (no value), jumper:JP1
- removed R4, R5: 220, rcl:0207/10
- removed T1: 2N3904, transistor:TO92
- added R2: (no value), pot:B25P
- C1, C2: value (none) -> 22p
- JP3: device jumper:JP2W -> jumper:JP2
- Q2: value (none) -> 16M
- moved JP7 153.6 mm to (41.9, 15.2)
- moved JP3 133.7 mm to (41.9, 21.6), turned to 270 degrees
- moved C4 133.1 mm to (8.89, 29.2)
- moved R6 96.5 mm to (20.3, 40.6)
- moved C3 96.1 mm to (8.89, 25.4)
- moved Q1 95.9 mm to (31.8, 27.9)
- moved C2 91.1 mm to (8.89, 21.6), turned to 180 degrees
- moved JP5 87.6 mm to (41.9, 7.62)
- moved LED1 84.8 mm to (40.6, 29.2)
- moved Q2 83.6 mm to (11.4, 14.0), turned to 270 degrees
- moved R1 83.6 mm to (38.1, 7.62), turned to 270 degrees
- moved C1 80.2 mm to (8.89, 6.35), turned to 180 degrees
- moved R8 76.1 mm to (6.35, 14.0), turned to 270 degrees
- moved R7 70.4 mm to (2.54, 14.0), turned to 270 degrees
- moved JP4 66.5 mm to (10.2, 2.54)
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Connections:
- removed net BJT_OUT: JP2.3, R5.2
- removed net LED_OUT: IC1.1, JP2.2
- removed net N$1: JP6.2, T1.1
- removed net N$6: JP6.1, R4.1
- removed net N$7: R5.1, T1.2
- new net MOSFET_GATE: Q1.1, R2.S
- net 12V: no longer R4.2
- net GND: now also R2.A; no longer T1.3
- net MOSFET_OUT: now also IC1.1, R2.E; no longer JP2.1, Q1.1
Routing:
- net GND: track 0.00 -> 153.7 mm, vias 0 -> 3
- net VCC: track 0.00 -> 93.7 mm, vias 0 -> 5
- net 12V: track 0.00 -> 49.9 mm, vias 0 -> 1
- net MOSFET_OUT: track 0.00 -> 35.9 mm, vias 0 -> 2
- net MOSFET_GATE: track 0.00 -> 34.4 mm, vias 0 -> 2
- net N$3: track 0.00 -> 27.5 mm, vias 0 -> 1
- net RX: track 0.00 -> 24.7 mm, vias 0 -> 2
- net N$9: track 0.00 -> 22.2 mm
- net N$4: track 0.00 -> 20.9 mm, vias 0 -> 1
- net IR_RX: track 0.00 -> 19.9 mm, vias 0 -> 1
- net +5V: track 0.00 -> 19.9 mm
- net XTAL1: track 0.00 -> 15.6 mm
- net XTAL2: track 0.00 -> 15.6 mm
- net N$8: track 0.00 -> 15.3 mm
- net N$2: track 0.00 -> 14.8 mm
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- added copper zone on layer 16, net N$1
- added copper zone on layer 1, net N$6
Other:
- board size 100 x 80 mm -> 45.4 x 43.2 mm
