File: Electronic Stuff/IR Module V2/IR_module_V0_2.sch (EAGLE design)
At the start: 24 parts, among them IC1 74HCT02N, Q1 IRF540, T1 2N3904

Commit message: IR module V0.2
Parts:
- removed JP2: (no value), jumper:JP2E
- removed JP6: (no value), jumper:JP1E
- removed R4, R5: 220, rcl:R-US_0207/10
- removed T1: 2N3904, transistor:2N3904
- added R2: (no value), pot:TRIM_US-B25P
- C1, C2: value (none) -> 22p
- JP3: device jumper:JP2W -> jumper:JP2E
- Q2: value (none) -> 16M
Connections:
- removed net BJT_OUT: JP2.3, R5.2
- removed net LED_OUT: IC1A.O, JP2.2
- removed net N$1: JP6.2, T1.C
- removed net N$6: JP6.1, R4.1
- removed net N$7: R5.1, T1.B
- new net MOSFET_GATE: Q1.G, R2.S
- net 12V: no longer R4.2
- net GND: now also R2.A; no longer T1.E
- net MOSFET_OUT: now also IC1A.O, R2.E; no longer JP2.1, Q1.G
