File: Electronic Stuff/IR Module V3/IR_module_V3.brd (EAGLE design)
At the start: 45.4 x 43.2 mm, 20 parts, among them IC1 74HCT02N, Q1 IRF540, Q2 16M

Commit message: IR
Connections:
- new net +5V: C3.2, ZU4.20, ZU4.7
- net VCC: no longer C3.2, ZU4.20, ZU4.7
Routing:
- net VCC: track 120.5 -> 93.7 mm
- net +5V: track 0.00 -> 19.9 mm
Changed lines of the file:
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@@
 <wire x1="43.18" y1="34.29" x2="34.29" y2="34.29" width="0.4064" layer="1"/>
 <wire x1="31.75" y1="24.13" x2="27.94" y2="24.13" width="0.4064" layer="16"/>
+</signal>
+<signal name="+5V" class="3">
 <contactref element="ZU4" pad="7"/>
+<contactref element="ZU4" pad="20"/>
 <contactref element="C3" pad="2"/>
-<contactref element="ZU4" pad="20"/>
 <wire x1="13.462" y1="25.4" x2="13.462" y2="24.638" width="0.4064" layer="16"/>
 <wire x1="13.462" y1="24.638" x2="13.97" y2="24.13" width="0.4064" layer="16"/>
@@
 <wire x1="17.78" y1="20.32" x2="22.86" y2="15.24" width="0.4064" layer="16"/>
 <wire x1="22.86" y1="15.24" x2="24.13" y2="15.24" width="0.4064" layer="16"/>
-<wire x1="24.13" y1="15.24" x2="25.4" y2="15.24" width="0.4064" layer="16"/>
-<wire x1="25.4" y1="15.24" x2="26.67" y2="16.51" width="0.4064" layer="16"/>
-<wire x1="26.67" y1="16.51" x2="30.48" y2="16.51" width="0.4064" layer="16"/>
 </signal>
 <signal name="RESET">
