File: Electronic Stuff/IR Module V3/IR_module_V3.brd (EAGLE design)
At the start: 45.4 x 43.2 mm, 20 parts, among them IC1 74HCT02N, Q1 IRF540, Q2 16M

Commit message: New PCB layout
Routing:
- net IR_RX: track 18.6 -> 17.3 mm
- net GND: track 152.5 -> 151.2 mm
Changed lines of the file:
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@@
 <wire x1="41.91" y1="29.21" x2="41.91" y2="26.67" width="0.4064" layer="16"/>
 <wire x1="41.91" y1="26.67" x2="39.37" y2="24.13" width="0.4064" layer="16"/>
-<wire x1="39.37" y1="24.13" x2="39.37" y2="20.32" width="0.4064" layer="16"/>
-<wire x1="39.37" y1="20.32" x2="40.64" y2="19.05" width="0.4064" layer="16"/>
 <wire x1="19.05" y1="11.43" x2="19.05" y2="16.51" width="0.4064" layer="16"/>
 <wire x1="19.05" y1="16.51" x2="17.78" y2="17.78" width="0.4064" layer="16"/>
@@
 <wire x1="19.05" y1="19.05" x2="19.05" y2="16.51" width="0.4064" layer="1"/>
 <contactref element="JP3" pad="2"/>
-<wire x1="39.37" y1="20.32" x2="41.91" y2="21.59" width="0" layer="19" extent="16-16"/>
+<wire x1="39.37" y1="24.13" x2="39.37" y2="22.86" width="0.4064" layer="16"/>
+<wire x1="39.37" y1="22.86" x2="40.64" y2="21.59" width="0.4064" layer="16"/>
+<wire x1="40.64" y1="21.59" x2="41.91" y2="21.59" width="0.4064" layer="16"/>
 </signal>
 <signal name="VCC">
@@
 <contactref element="IC1" pad="12"/>
 <wire x1="38.1" y1="10.16" x2="35.56" y2="12.7" width="0.4064" layer="16"/>
-<wire x1="40.64" y1="21.59" x2="39.37" y2="20.32" width="0.4064" layer="1"/>
-<wire x1="39.37" y1="20.32" x2="39.37" y2="13.97" width="0.4064" layer="1"/>
 <wire x1="39.37" y1="13.97" x2="40.64" y2="12.7" width="0.4064" layer="1"/>
 <wire x1="40.64" y1="12.7" x2="40.64" y2="11.43" width="0.4064" layer="1"/>
@@
 <wire x1="40.64" y1="10.16" x2="40.64" y2="11.43" width="0.4064" layer="16"/>
 <contactref element="JP3" pad="3"/>
-<wire x1="40.64" y1="21.59" x2="41.91" y2="19.05" width="0" layer="19" extent="1-1"/>
+<wire x1="39.37" y1="13.97" x2="39.37" y2="17.78" width="0.4064" layer="1"/>
+<wire x1="39.37" y1="17.78" x2="40.64" y2="19.05" width="0.4064" layer="1"/>
+<wire x1="40.64" y1="19.05" x2="41.91" y2="19.05" width="0.4064" layer="1"/>
 </signal>
 <signal name="N$8">
