File: Electronic Stuff/IR Module V3/IR_module_V3.sch (EAGLE design)
At the start: 20 parts, among them IC1 74HCT02N, Q1 IRF540, Q2 16M

Commit message: IR
Connections:
- new net +5V: C3.2, ZU4.AVCC, ZU4.VCC
- net VCC: no longer C3.2, ZU4.AVCC, ZU4.VCC
Changed lines of the file:
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@@
 <parts>
 <part name="ZU4" library="SmartPrj" deviceset="ATMEGA328P-" device="PU"/>
+<part name="P+3" library="supply1" deviceset="+5V" device=""/>
 <part name="GND2" library="supply1" deviceset="GND" device=""/>
 <part name="GND3" library="supply1" deviceset="GND" device=""/>
@@
 <part name="R2" library="pot" deviceset="TRIM_US-" device="B25P"/>
 <part name="GND10" library="supply1" deviceset="GND" device=""/>
-<part name="P+3" library="supply1" deviceset="VCC" device=""/>
 </parts>
 <sheets>
@@
 <instances>
 <instance part="ZU4" gate="G$1" x="157.48" y="53.34"/>
+<instance part="P+3" gate="1" x="119.38" y="53.34" smashed="yes">
+<attribute name="VALUE" x="121.285" y="55.88" size="1.778" layer="96" rot="R180"/>
+</instance>
 <instance part="GND2" gate="1" x="129.54" y="33.02"/>
 <instance part="GND3" gate="1" x="99.06" y="66.04"/>
@@
 <instance part="R2" gate="G$1" x="284.48" y="60.96"/>
 <instance part="GND10" gate="1" x="284.48" y="48.26"/>
-<instance part="P+3" gate="VCC" x="119.38" y="55.88"/>
 </instances>
 <busses>
 </busses>
 <nets>
+<net name="+5V" class="3">
+<segment>
+<wire x1="137.16" y1="50.8" x2="124.46" y2="50.8" width="0.1524" layer="91"/>
+<pinref part="ZU4" gate="G$1" pin="VCC"/>
+<pinref part="P+3" gate="1" pin="+5V"/>
+<pinref part="ZU4" gate="G$1" pin="AVCC"/>
+<wire x1="124.46" y1="50.8" x2="119.38" y2="50.8" width="0.1524" layer="91"/>
+<wire x1="137.16" y1="58.42" x2="124.46" y2="58.42" width="0.1524" layer="91"/>
+<wire x1="124.46" y1="58.42" x2="124.46" y2="50.8" width="0.1524" layer="91"/>
+<pinref part="C3" gate="G$1" pin="2"/>
+<wire x1="124.46" y1="48.26" x2="124.46" y2="50.8" width="0.1524" layer="91"/>
+</segment>
+</net>
 <net name="GND" class="2">
 <segment>
@@
 <wire x1="307.34" y1="38.1" x2="312.42" y2="38.1" width="0.1524" layer="91"/>
 </segment>
-<segment>
-<wire x1="137.16" y1="50.8" x2="124.46" y2="50.8" width="0.1524" layer="91"/>
-<pinref part="ZU4" gate="G$1" pin="VCC"/>
-<pinref part="ZU4" gate="G$1" pin="AVCC"/>
-<wire x1="124.46" y1="50.8" x2="119.38" y2="50.8" width="0.1524" layer="91"/>
-<wire x1="137.16" y1="58.42" x2="124.46" y2="58.42" width="0.1524" layer="91"/>
-<wire x1="124.46" y1="58.42" x2="124.46" y2="50.8" width="0.1524" layer="91"/>
-<pinref part="C3" gate="G$1" pin="2"/>
-<wire x1="124.46" y1="48.26" x2="124.46" y2="50.8" width="0.1524" layer="91"/>
-<pinref part="P+3" gate="VCC" pin="VCC"/>
-<wire x1="119.38" y1="50.8" x2="119.38" y2="53.34" width="0.1524" layer="91"/>
-</segment>
-</net>
+</net>
