File: Electronic Stuff/IR Module V3/IR_module_V3.sch (EAGLE design)
At the start: 20 parts, among them IC1 74HCT02N, Q1 IRF540, Q2 16M

Commit message: Added texts
Parts:
- C1, C2, C3, C4: device SparkFun-Passives:CAPPTH3 -> SparkFun-Capacitors:CAPEZ
Changed lines of the file:
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@@
 <part name="R8" library="rcl" deviceset="R-US_" device="0207/10" value="1M"/>
 <part name="Q2" library="crystal" deviceset="CRYSTAL" device="HC49S" value="16M"/>
-<part name="C1" library="SparkFun-Passives" deviceset="CAP" device="PTH3" value="22p"/>
-<part name="C2" library="SparkFun-Passives" deviceset="CAP" device="PTH3" value="22p"/>
-<part name="C3" library="SparkFun-Passives" deviceset="CAP" device="PTH3" value="100n"/>
+<part name="C1" library="SparkFun-Capacitors" deviceset="CAP" device="EZ" value="22p"/>
+<part name="C2" library="SparkFun-Capacitors" deviceset="CAP" device="EZ" value="22p"/>
+<part name="C3" library="SparkFun-Capacitors" deviceset="CAP" device="EZ" value="100n"/>
 <part name="JP3" library="jumper" deviceset="JP2E" device=""/>
 <part name="JP7" library="jumper" deviceset="JP1E" device=""/>
 <part name="P+4" library="supply1" deviceset="VCC" device=""/>
 <part name="GND12" library="supply1" deviceset="GND" device=""/>
-<part name="C4" library="SparkFun-Passives" deviceset="CAP" device="PTH3" value="100n"/>
+<part name="C4" library="SparkFun-Capacitors" deviceset="CAP" device="EZ" value="100n"/>
 <part name="R2" library="pot" deviceset="TRIM_US-" device="B25P"/>
 <part name="GND10" library="supply1" deviceset="GND" device=""/>
